Commit message: backup

File: src/my_learning_package/urdf/AionR1.urdf.xacro (robot description, xacro)
@@ -2,9 +2,10 @@
 <robot xmlns:xacro="http://www.ros.org/wiki/xacro" name="aion_r1">
     <xacro:include filename="inertial_macros.xacro"/>
+    <!-- <xacro:include filename="materials.urdf.xacro"/> -->
 <!-- <?xml version="1.0" ?>
 <sdf version="1.5"> -->
   <!-- <model name="aion_robotics_r1_rover"> -->
     <!-- MATERIALS / COLOURS -->
-    <material name="white">
+    <!-- <material name="white">
         <color rgba="1 1 1 1"/>
     </material>
@@ -14,5 +15,5 @@
     <material name="black">
         <color rgba="0 0 0 1"/>
-    </material>
+    </material> -->
     <link name="aion_base_link">
         <collision>

File: src/my_learning_package/urdf/loam_robot_01.urdf.xacro (robot description, xacro)
@@ -1,10 +1,12 @@
 <?xmm version="1.0"?>
 <robot xmlns:xacro="http://www.ros.org/wiki/xacro" name="loam_robot_01">
-    <material name="light_brown" >
+    <!-- <material name="light_brown" >
         <color rgba="1.0 0.9 0.6 1" />
-    </material>
+    </material> -->
+    <xacro:include filename="materials.urdf.xacro"/>
     <!-- include lidar mid 70 -->
     <xacro:include filename="mid70.urdf.xacro"/>
     <xacro:include filename="MTi_10.urdf.xacro"/>
+    <xacro:include filename="materials.urdf.xacro"/>
     <link name="base_link">
     </link>

File: src/my_learning_package/urdf/mid70.urdf.xacro (robot description, xacro)
@@ -2,21 +2,32 @@
 <robot xmlns:xacro="http://www.ros.org/wiki/xacro" >
     <xacro:include filename="inertial_macros.xacro"/>
+    <!-- <xacro:include filename="materials.urdf.xacro"/> -->
     <!-- color of lidar, TODO: put colors into separate xacro file -->
-    <material name="light_gray" >
+    <!-- <material name="light_gray" >
         <color rgba="0.8 0.8 0.8 1" />
-    </material>
+    </material> -->
     <link name="livox_frame" >
         <visual>
-            <origin xyz="-0.0323 0 -0.00105"/> <!-- x = 0.097/2 - 0.0162  z = 0.0627/2 - 0.0324, from manual of mid70, see center point location page 15-->
+            <!-- <origin xyz="-0.0323 0 -0.00105"/> x = 0.097/2 - 0.0162  z = 0.0627/2 - 0.0324, from manual of mid70, see center point location page 15 -->
+            <origin xyz="-0.0659 0 0" rpy="${0} ${pi/2} ${-pi/2}"/>
+            <!-- <geometry>
+                <box size="0.097 0.064 0.0627" />
+            </geometry> -->
             <geometry>
-                <box size="0.097 0.064 0.0627" />
+                <!-- <mesh filename="file:///home/slamnuc/ros2_learning_ws/src/my_learning_package/urdf/MTi_10.stl" scale="0.001 0.001 0.001"/> -->
+                <mesh filename="package://my_learning_package/urdf/livox_mid-70_nocone.stl" scale="0.001 0.001 0.001"/>
             </geometry>
             <material name="light_gray" />
         </visual>
         <collision>
-            <origin xyz="-0.0323 0 -0.00105"/> <!-- x = 0.097/2 - 0.0162  z = 0.0627/2 - 0.0324, from manual of mid70, see center point location page 15-->
+            <!-- <origin xyz="-0.0323 0 -0.00105"/> x = 0.097/2 - 0.0162  z = 0.0627/2 - 0.0324, from manual of mid70, see center point location page 15 -->
+            <origin xyz="-0.0659 0 0" rpy="${0} ${pi/2} ${-pi/2}"/>
             <geometry>
+                <!-- <mesh filename="file:///home/slamnuc/ros2_learning_ws/src/my_learning_package/urdf/MTi_10.stl" scale="0.001 0.001 0.001"/> -->
+                <mesh filename="package://my_learning_package/urdf/livox_mid-70_nocone.stl" scale="0.001 0.001 0.001"/>
+            </geometry>
+            <!-- <geometry>
                 <box size="0.097 0.064 0.0627" />
-            </geometry>
+            </geometry> -->
         </collision>
         <xacro:inertial_box mass="0.580" x="0.097" y="0.064" z="0.0627">
@@ -24,3 +35,8 @@
         </xacro:inertial_box>
     </link>
+    <!-- <joint name="lidar_odom_joint" type="fixed">
+        <parent link="livox_frame"/>
+        <child link="lidar_odom"/>
+        <origin xyz="0 0 0"/>
+    </joint>  -->
 </robot>
