Commit message: backup

File: src/my_learning_package/urdf/data_platform.urdf.xacro (robot description, xacro)
@@ -10,22 +10,119 @@
     <!-- <xacro:include filename="materials.urdf.xacro"/> -->
     <!-- <xacro:include filename="AionR1.urdf.xacro"/> -->
+    <!-- main wooden platform -->
     <link name="data_platform_base_link" >
         <visual>
-            <origin xyz="0 0 0"/> <!-- x = 0.097/2 - 0.00162  z = 0.0627/2 - 0.0324, from manual of mid70, see center point location page 15-->
+            <origin xyz="0 0 -0.0015"/> <!-- x = 0.097/2 - 0.00162  z = 0.0627/2 - 0.0324, from manual of mid70, see center point location page 15-->
             <geometry>
-                <box size="0.30 0.343 0.003" />
+                <box size="0.394 0.23 0.003" />
             </geometry>
             <material name="light_brown" />
         </visual>
     </link>
+    <link name="nuc" >
+        <visual>
+            <origin xyz="0.0551 0.02505 0.0551"/>
+            <geometry>
+                <box size="0.112 0.051 0.112"/>
+            </geometry>
+            <material name="black"/>
+        </visual>
+    </link>
+    <joint name="nuc_joint" type="fixed">
+        <parent link="data_platform_base_link"/>
+        <child link="nuc"/>  <!--  TODO: correct to livox_base-->
+        <origin xyz="0.0468 0.115 -0.041"/>  <!-- see mid-70 documentation for center of origin of lidar-->
+    </joint>
     <joint name="lidar_joint" type="fixed">
         <parent link="data_platform_base_link"/>
-        <child link="livox_frame"/>  <!--  TODO: need to rename the frame of the lidar at some point..-->
-        <origin xyz="0.15 0 0.04"/>
+        <child link="livox_base"/>  <!--  TODO: correct to livox_base-->
+        <origin xyz="0.100 0 0.0"/>  <!-- see mid-70 documentation for center of origin of lidar-->
     </joint>
     <!-- small plywood plate on top of lidar connection the imu to lidar -->
-    <link name="mounting_plate" >
+    <!-- x = 0.097/2 - 0.00162  z = 0.0627/2 - 0.0324, from manual of mid70, see center point location page 15-->
+    <link name="mounting_plate_bottom" >
         <visual>
-            <origin xyz="0 0 0"/> <!-- x = 0.097/2 - 0.00162  z = 0.0627/2 - 0.0324, from manual of mid70, see center point location page 15-->
+            <origin xyz="0 0 -0.0015"/> <!-- x = 0.097/2 - 0.00162  z = 0.0627/2 - 0.0324, from manual of mid70, see center point location page 15-->
+            <geometry>
+                <box size="0.10 0.078 0.003" />
+            </geometry>
+            <material name="light_brown" />
+        </visual>
+        <visual>
+            <origin xyz="0.0305 0.023 -0.008"/>
+            <geometry>
+                <cylinder radius="0.00235" length="0.01"/>
+            </geometry>
+        </visual>
+        <visual>
+            <origin xyz="0.0305 -0.023 -0.008"/>
+            <geometry>
+                <cylinder radius="0.00235" length="0.01"/>
+            </geometry>
+        </visual>
+        <visual>
+            <origin xyz="-0.0305 0.023 -0.008"/>
+            <geometry>
+                <cylinder radius="0.00235" length="0.01"/>
+            </geometry>
+        </visual>
+        <visual>
+            <origin xyz="-0.0305 -0.023 -0.008"/>
+            <geometry>
+                <cylinder radius="0.00235" length="0.01"/>
+            </geometry>
+        </visual>
+    </link>
+    <joint name="mounting_plate_dampening_joint" type="fixed">
+        <parent link="mounting_plate_bottom"/>
+        <child link="mounting_plate_top" />
+        <origin xyz="0.0 0 0.015"/>
+    </joint>
+    <link name="mounting_plate_top" >
+        <visual>
+            <origin xyz="0 0 -0.0015"/> <!-- x = 0.097/2 - 0.00162  z = 0.0627/2 - 0.0324, from manual of mid70, see center point location page 15-->
+            <geometry>
+                <box size="0.10 0.078 0.003" /> <!-- old dimensions 0.0708 0.0596 0.003-->
+            </geometry>
+            <material name="light_brown" />
+        </visual>
+    </link>
+    <joint name="mounting_plate_top_dampening_spacers" type="fixed">
+        <parent link="mounting_plate_top"/>
+        <child link="dampening_rubber_spacers" />
+        <origin xyz="0 0 -0.0015"/>
+    </joint>
+    <link name="dampening_rubber_spacers" >
+        <visual>
+            <material name="blue" />
+            <origin xyz="0.04 0 -0.0075"/> <!-- x = 0.097/2 - 0.00162  z = 0.0627/2 - 0.0324, from manual of mid70, see center point location page 15-->
+            <geometry>
+                <sphere radius="0.0088"/>
+            </geometry>
+        </visual>
+        <visual>
+            <material name="blue" />
+            <origin xyz="-0.025 0.0305 -0.0075"/> <!-- x = 0.097/2 - 0.00162  z = 0.0627/2 - 0.0324, from manual of mid70, see center point location page 15-->
+            <geometry>
+                <sphere radius="0.0088"/>
+            </geometry>
+        </visual>
+        <visual>
+            <material name="blue" />
+            <origin xyz="-0.025 -0.0305 -0.0075"/> <!-- x = 0.097/2 - 0.00162  z = 0.0627/2 - 0.0324, from manual of mid70, see center point location page 15-->
+            <geometry>
+                <sphere radius="0.0088"/>
+            </geometry>
+        </visual>
+    </link>
+    <joint name="mounting_plate_joint" type="fixed">
+        <parent link="livox_frame"/>
+        <child link="mounting_plate_bottom" />
+        <origin xyz="-0.04275 0 0.0433"/>
+    </joint>
+    <!-- needs to be fitted -->
+    <!-- <link name="mounting_plate_with_dampening" >
+        <visual>
+            <origin xyz="0 0 0"/>
             <geometry>
                 <box size="0.0708 0.0596 0.003" />
@@ -33,14 +130,22 @@
             <material name="light_brown" />
         </visual>
+    </link> -->
+    <!-- needs to be fitted -->
+    <!-- <joint name="mounting_plate_joint" type="fixed">
+        <parent link="livox_frame"/>
+        <child link="mounting_plate_with_dampening" />
+        <origin xyz="-0.04275 0 0.0318"/>
+    </joint> -->
+    <!-- <link name="lidar_odom" >
     </link>
-    <joint name="mounting_plate_joint" type="fixed">
+    <joint name="livox_frame_to_lidar_odom" type="fixed">
         <parent link="livox_frame"/>
-        <child link="mounting_plate" />
-        <origin xyz="-0.04275 0 0.0318"/>
-    </joint>
+        <child link="lidar_odom" />
+        <origin xyz="0 0 0"/>
+    </joint> -->
     <joint name="imu_joint" type="fixed">
-        <parent link="mounting_plate"/>
+        <parent link="mounting_plate_top"/>
         <child link="imu_base_link" />
-        <origin xyz="-0.0246 0.017 0.0015"/>
+        <origin xyz="-0.0246 0.017 0.0"/>
     </joint>
 </robot>

File: src/my_learning_package/urdf/loam_robot_viz.urdf.xacro (robot description, xacro)
@@ -18,8 +18,9 @@
         <origin xyz="-0.20 0 0"/>
     </joint>
+    <!-- subtract 1 mm to z for the Aion top plate thicknes -->
     <joint name="data_platform_joint" type="fixed">
         <parent link="top_plate_link"/>
         <child link="data_platform_base_link" />
-        <origin xyz="0 0 0.05"/>
+        <origin xyz="0 0 0.0447"/>
     </joint>
     <!-- <joint name="lidar_odom_joint" type="fixed">

File: src/my_learning_package/urdf/materials.urdf.xacro (robot description, xacro)
@@ -16,3 +16,6 @@
         <color rgba="0 0 0 1"/>
     </material>
+    <material name="blue">
+        <color rgba="0 0 1 1"/>
+    </material>
 </robot>

File: src/my_learning_package/urdf/mid70.urdf.xacro (robot description, xacro)
@@ -7,4 +7,12 @@
         <color rgba="0.8 0.8 0.8 1" />
     </material> -->
+    <!-- low back edge in the center line -->
+    <link name="livox_base">
+    </link>
+    <joint name="livox_base_to_frame" type="fixed">
+        <parent link="livox_base"/>
+        <child link="livox_frame"/>
+        <origin xyz="0.0794 0 0.0324"/>  <!--x 0.0794, should be 97 -16.2 = 80.2 mm? y 0 z 0.0324 -->
+    </joint>
     <link name="livox_frame" >
         <visual>
